Commit message: Added Robot Description, Gazebo and Localization packages

File: src/robot_description/urdf/robot.camera.xacro (robot description, xacro)
@@ -2,30 +2,42 @@
 <robot xmlns:xacro="http://www.ros.org/wiki/xacro">
   <xacro:macro
-    name="robby_camera"
+    name="robot_camera"
     params="
       parent:=chassis_link
-      xyz:='0.12 0 0.18'
+      xyz:='0.15 0.0 0.0195'
       rpy:='0 0 0'
       add_gazebo:=false
-      topic:=/camera/image_raw
-      update_rate:=15.0
-      width:=640
-      height:=480
-      hfov:=1.39626
-      near_clip:=0.05
-      far_clip:=20.0">
+      topic:=/camera
+      update_rate:=30.0
+      width:=1280
+      height:=720
+      hfov:=1.5184
+      vfov:=1.0122
+      near_clip:=0.07
+      far_clip:=6.0
+      stereo_baseline:=0.018
+      dimension_x:=0.042
+      dimension_y:=0.042
+      dimension_z:=0.023
+      ">
     <link name="camera_link">
       <inertial>
         <origin xyz="0 0 0" rpy="0 0 0" />
-        <mass value="0.12" />
-        <inertia ixx="8e-5" ixy="0.0" ixz="0.0" iyy="8e-5" iyz="0.0" izz="8e-5" />
+        <mass value="0.0387416202428435" />
+        <inertia
+          ixx="1.08456634317136E-05"
+          ixy="0.0"
+          ixz="0.0"
+          iyy="7.10436611069618E-06"
+          iyz="0.0"
+          izz="7.1103467824982E-06" />
       </inertial>
       <visual>
         <origin xyz="0 0 0" rpy="0 0 0" />
         <geometry>
-          <box size="0.05 0.04 0.035" />
+          <mesh filename="package://robot_description/meshes/camera_link.STL" />
         </geometry>
-        <material name="camera_black">
-          <color rgba="0.08 0.08 0.08 1.0" />
+        <material name="camera_body">
+          <color rgba="0.05 0.12 0.55 1" />
         </material>
       </visual>
@@ -33,5 +45,5 @@
         <origin xyz="0 0 0" rpy="0 0 0" />
         <geometry>
-          <box size="0.05 0.04 0.035" />
+          <box size="0.023 0.0421 0.0420" />
         </geometry>
       </collision>
@@ -56,5 +68,6 @@
     <xacro:if value="${add_gazebo}">
       <gazebo reference="camera_link">
-        <sensor name="camera_sensor" type="camera">
+        <material>Gazebo/Blue</material>
+        <sensor name="camera_sensor" type="rgbd_camera">
           <always_on>1</always_on>
           <update_rate>${update_rate}</update_rate>

File: src/robot_description/urdf/robot.core.xacro (robot description, xacro)
@@ -85,5 +85,5 @@
     </joint>
   </xacro:macro>
-  <xacro:macro name="robby_robot" params="mesh_dir">
+  <xacro:macro name="robot_robot" params="mesh_dir">
     <xacro:property name="mesh_uri_root" value="${mesh_dir}" />
     <xacro:property name="front_steer_limit" value="1.5708" />

File: src/robot_description/urdf/robot.gazebo.xacro (robot description, xacro)
@@ -1,5 +1,5 @@
 <?xml version="1.0" encoding="utf-8"?>
-<robot xmlns:xacro="http://www.ros.org/wiki/xacro" name="Robby_v1">
-  <xacro:arg name="mesh_dir" default="package://robby_description/meshes" />
+<robot xmlns:xacro="http://www.ros.org/wiki/xacro" name="robot">
+  <xacro:arg name="mesh_dir" default="package://robot_description/meshes" />
   <xacro:arg name="controllers_file" default="" />
   <xacro:arg name="imu_update_rate" default="100.0" />
@@ -14,7 +14,7 @@
   <xacro:arg name="camera_topic" default="/camera/image_raw" />
   <xacro:arg name="camera_update_rate" default="15.0" />
-  <xacro:include filename="Robby_v1.core.xacro" />
-  <xacro:include filename="Robby_v1.lidar.xacro" />
-  <xacro:include filename="Robby_v1.camera.xacro" />
+  <xacro:include filename="robot.core.xacro" />
+  <xacro:include filename="robot.lidar.xacro" />
+  <xacro:include filename="robot.camera.xacro" />
   <xacro:macro name="ros2_control_position_joint" params="joint_name">
     <joint name="${joint_name}">
@@ -31,7 +31,7 @@
     </joint>
   </xacro:macro>
-  <xacro:robby_robot mesh_dir="$(arg mesh_dir)" />
+  <xacro:robot_robot mesh_dir="$(arg mesh_dir)" />
   <xacro:if value="$(arg use_lidar)">
-    <xacro:robby_lidar
+    <xacro:robot_lidar
       parent="chassis_link"
       xyz="$(arg lidar_xyz)"
@@ -42,5 +42,5 @@
   </xacro:if>
   <xacro:if value="$(arg use_camera)">
-    <xacro:robby_camera
+    <xacro:robot_camera
       parent="chassis_link"
       xyz="$(arg camera_xyz)"
@@ -57,5 +57,5 @@
     </sensor>
   </gazebo>
-  <ros2_control name="RobbyGazeboSystem" type="system">
+  <ros2_control name="robotGazeboSystem" type="system">
     <hardware>
       <plugin>gz_ros2_control/GazeboSimSystem</plugin>

File: src/robot_description/urdf/robot.lidar.xacro (robot description, xacro)
@@ -2,5 +2,5 @@
 <robot xmlns:xacro="http://www.ros.org/wiki/xacro">
   <xacro:macro
-    name="robby_lidar"
+    name="robot_lidar"
     params="
       parent:=chassis_link

File: src/robot_description/urdf/robot.urdf.xacro (robot description, xacro)
@@ -1,6 +1,6 @@
 <?xml version="1.0" encoding="utf-8"?>
-<!-- Clean robot description only. Gazebo and ros2_control live in Robby_v1.gazebo.xacro. -->
-<robot xmlns:xacro="http://www.ros.org/wiki/xacro" name="Robby_v1">
-  <xacro:arg name="mesh_dir" default="package://robby_description/meshes" />
+<!-- Clean robot description only. Gazebo and ros2_control live in robot.gazebo.xacro. -->
+<robot xmlns:xacro="http://www.ros.org/wiki/xacro" name="robot">
+  <xacro:arg name="mesh_dir" default="package://robot_description/meshes" />
   <xacro:arg name="use_lidar" default="false" />
   <xacro:arg name="lidar_xyz" default="0 0 0.15" />
@@ -9,10 +9,10 @@
   <xacro:arg name="camera_xyz" default="0.12 0 0.18" />
   <xacro:arg name="camera_rpy" default="0 0 0" />
-  <xacro:include filename="Robby_v1.core.xacro" />
-  <xacro:include filename="Robby_v1.lidar.xacro" />
-  <xacro:include filename="Robby_v1.camera.xacro" />
-  <xacro:robby_robot mesh_dir="$(arg mesh_dir)" />
+  <xacro:include filename="robot.core.xacro" />
+  <xacro:include filename="robot.lidar.xacro" />
+  <xacro:include filename="robot.camera.xacro" />
+  <xacro:robot_robot mesh_dir="$(arg mesh_dir)" />
   <xacro:if value="$(arg use_lidar)">
-    <xacro:robby_lidar
+    <xacro:robot_lidar
       parent="chassis_link"
       xyz="$(arg lidar_xyz)"
@@ -21,5 +21,5 @@
   </xacro:if>
   <xacro:if value="$(arg use_camera)">
-    <xacro:robby_camera
+    <xacro:robot_camera
       parent="chassis_link"
       xyz="$(arg camera_xyz)"
