Commit message: GripperX: third full sync from the working repo (2026-08-25 -> 2026-09-23)
Four weeks since the second sync. 99 files change, 4 are new, and the export
shrinks by roughly 800 lines on balance -- that is a comment-slimming pass, not
lost function. Nothing outside GripperX/ is touched.

WHAT IS NEW, IN THE ORDER IT MATTERS

  * Navigation rotation is repaired, and it is the largest change here. Four
    separate defects, each merged and measured on its own: the local costmap
    never saw the map SLAM had already built (59 of 72 rejections were
    "Trajectory Hits Unknown Region"); the stall detector latched motors off
    during the alignment gate's own legitimate hold; in-place rotation shared a
    controller with path following and sampled inside a band the steering
    limiter silently widens; and bt_navigator ran a 20 ms acknowledgement budget
    its own tick loop cannot resolve, so a 15-20 ms acknowledgement was never
    read. Measured on the robot between 2026-09-15 and 2026-09-23: goals reached
    5/37 -> 8/10, "No valid trajectories" 118 -> 0, stall latches 17 -> 0,
    acknowledgement timeouts 2/10 -> 0/10. Deployed and endorsed, NOT signed off
    item by item -- read the numbers as measurements, not as an acceptance.

  * The steering alignment timing invariant was broken for 27 days and is fixed.
    The controller's alignment timeout was raised 1.5 -> 5.0 s on 2026-08-25 and
    the gate enabled the same day; the navigation-side grace that has to exceed
    it stayed at 2.0 s, so every sideways-swerve recovery failed by
    construction. Grace is now 5.5 s, and gripperx_control/test/
    check_alignment_timing.py parses both YAML files and fails if the relation
    inverts again. The two values live in different files and different nodes,
    which is why nothing caught it for four weeks.

  * The steering couplings were rebuilt in ASA and all four wheels recalibrated.
    Measured effect over repeated identical crab manoeuvres: yaw spread fell
    16.73 -> 2.08 degrees, a factor of eight, against a prediction recorded
    before the runs. The outward steering limit moved 100 -> 125 degrees, and
    the executing constants that still carried 100 were found and corrected --
    two diagnostic tools that command drive and steering were among them.

  * The clean-shutdown button is accepted on the robot. Ten short presses, each
    approved individually, verified per node. A short press restarts the ROS
    stack and leaves the computer up; a long press shuts down; 1-3 seconds is a
    deliberate dead zone that discards the press. Note the button gives no
    feedback, so a discarded press is indistinguishable from a dead button.

  * The desk launcher now opens the browser teleop by default (--keyboard is the
    escape hatch), and its real-robot mode is verified including the browser
    front-end.

WHAT SHRANK, AND WHY IT IS SAFE

A comment-slimming pass went through the source tree: the chronicle of how each
file reached its current state is removed, while every comment that protects the
next edit -- an invariant, a measured value, a trap -- is kept. No logic
changed. Where a comment turned out to state something the configuration
refutes, the comment was corrected rather than deleted; the 125 degree steering
limit is the clearest case, where the stated rationale had been carried forward
from a calibration the rework replaced.

TWO THINGS TO KNOW WHEN READING THE CODE

  * Geometry has exactly one home: gripperx_geometry/config/geometry.yaml.
    Changing a wheel radius or track width anywhere else will disagree with the
    rest of the stack. This is unchanged from the last sync and still the most
    common way to break something quietly.
  * A few comments name internal records that are not part of this repository --
    the working repo keeps a requirements document and analysis notes that the
    export does not carry. New files name them in words; five older references
    still cite them by path and are owed a cleanup.

File: GripperX/Software/ros2/src/gripperx_description/urdf/gripperx_v1.core.xacro (robot description, xacro)
@@ -89,9 +89,10 @@
   <xacro:macro name="gripperx_robot" params="mesh_dir">
     <xacro:property name="mesh_uri_root" value="${mesh_dir}" />
-    <!-- STEERING WINDOW — asymmetric and per wheel (calibrated on the machine
-         2026-08-13; source of truth: gripperx_control/config/steer_servo.yaml).
-         Every wheel reaches ~100 deg OUTWARD (tyre swings away from the chassis)
-         and only ~30 deg INWARD, and which SIGN of the joint angle is outward
-         differs per wheel — MEASURED as [-1,+1,+1,-1] for FL, FR, BL, BR. It is
+    <!-- STEERING WINDOW — asymmetric and per wheel (source of truth:
+         gripperx_control/config/steer_servo.yaml; current values recalibrated
+         2026-09-18). Every wheel reaches an outward limit far larger than the
+         inward one (see the table below for the current figures), and which
+         SIGN of the joint angle is outward differs per wheel — MEASURED as
+         [-1,+1,+1,-1] for FL, FR, BL, BR. It is
          NOT derivable from this model: each wheel hangs on a lateral lever arm
          off its king pin (*_wheel_offset_xyz, y = +-0.0556 m), so turning the
@@ -105,20 +106,32 @@
          rounds. A stale value left in prose is exactly how it hid.
          Resulting joint windows (all four joints turn about base_link +Z, so
-         +angle points a wheel to the robot's left):
-             f_left_steer   [-100, +30]      b_leftsteer   [-30, +100]
-             f_right_steer  [ -30, +100]     b_rightsteer  [-100, +30]  deg
+         +angle points a wheel to the robot's left; current values, see
+         steer_servo.yaml):
+             f_left_steer   [-125, +35]      b_leftsteer   [-35, +125]
+             f_right_steer  [ -35, +125]     b_rightsteer  [-125, +35]  deg
          This is the digital twin's model too: the twin must not be able to reach
          a pose the real robot cannot, so these are the real limits and NOT a
          relaxed sim variant. The former symmetric front_steer_limit /
          rear_steer_limit (1.0472 = 60 deg both ways) is gone — it allowed the
-         twin 60 deg inward, twice what the mechanics has, while wasting 40 deg
-         of the outward travel. The in-place spin pose (+-58.57 deg, outward on
-         all four) still fits comfortably. -->
-    <xacro:property name="steer_outward_limit" value="1.745329" />
+         twin more inward travel than the mechanics has, while wasting outward
+         travel. The in-place spin pose (+-58.57 deg, outward on all four) still
+         fits comfortably. -->
+    <xacro:property name="steer_outward_limit" value="2.181662" />
     <xacro:property name="steer_inward_limit" value="0.610865" />
-    <!-- inward 30 -> 35 deg (0.523599 -> 0.610865) on 2026-08-18, tracking
-         gripperx_control/config/steer_servo.yaml (source of truth). Both the
-         35 deg limit and the inward travel it sits in are TO-VERIFY - see the
-         unresolved inward-stop contradiction documented in that file. -->
+    <!-- outward 100 -> 125 deg (1.745329 -> 2.181662) on 2026-09-18, inward
+         30 -> 35 deg (0.523599 -> 0.610865) on 2026-08-18, both tracking
+         gripperx_control/config/steer_servo.yaml (source of truth). The
+         inward-stop contradiction that made these TO-VERIFY is RESOLVED: the
+         stops were re-measured at the real mechanical limit on 2026-09-18 and
+         the tightest inward travel is 50.3 deg, so 35 deg sits on 15.3 deg of
+         margin rather than the ~0.6 deg once feared. 125 deg outward is a
+         chosen working margin, not a value derived from a hard constraint: it
+         leaves roughly 70 deg to the measured mechanical stop (193.6-196.4 deg
+         on the tightest wheel) and stays short of the angle where the left and
+         right wheel could touch in an unfavourable combination. CORRECTED
+         2026-09-23: this comment previously said 125 was bound by FL's
+         raw-count wrap — wrong twice over, see gripperx_control's
+         steering_limits.py for the full correction; the mechanical stop binds
+         long before any wrap. -->
     <xacro:property name="joint_effort" value="10" />
     <xacro:property name="joint_velocity" value="10" />
